Commit message: Add mujoco replay to gui && add annotation && Improve data collection GUI replay safety

File: src/lerobot/robots/franka_research3/assets/franka_fr3/fr3_pika_gripper_ati.urdf (robot description, URDF)
Before this commit: robot fr3, 17 links, 16 joints
Links:
- added link pika_task_tcp
Joints:
- added joint pika_task_tcp_joint: type fixed, parent gripper_base_link, child pika_task_tcp, origin xyz=0 0 0.366842 rpy=3.1415926 -1.5707963 0

Commit message: add fr3 corenetic urdf and mujoco xml

File: src/lerobot/robots/franka_research3/assets/franka_fr3/fr3_pika_gripper_ati.urdf (robot description, URDF)
Before this commit: robot fr3, 18 links, 17 joints
Joints:
- joint fr3_hand_tcp_joint: type fixed -> revolute
