Commit message: add teleop workstation pipeline

File: src/lerobot/robots/franka_research3/assets/franka_fr3/fr3_pika_gripper.urdf (robot description, URDF)
Before this commit: robot fr3, 14 links, 13 joints
Links:
- added link fr3_pika_adapter_link, mass 0.0192; collision mesh filename=./assets/fr32pika.STL scale=0.001 0.001 0.001; visual mesh filename=./assets/fr32pika.STL scale=0.001 0.001 0.001
- added link pika_task_tcp
- link fr3_link0: geometry collision mesh filename=./assets/fr3/collision/link0.stl; visual mesh filename=./assets/fr3/visual/link0.dae
- link fr3_link1: geometry collision mesh filename=./assets/fr3/collision/link1.stl; visual mesh filename=./assets/fr3/visual/link1.dae
- link fr3_link2: geometry collision mesh filename=./assets/fr3/collision/link2.stl; visual mesh filename=./assets/fr3/visual/link2.dae
- link fr3_link3: geometry collision mesh filename=./assets/fr3/collision/link3.stl; visual mesh filename=./assets/fr3/visual/link3.dae
- link fr3_link4: geometry collision mesh filename=./assets/fr3/collision/link4.stl; visual mesh filename=./assets/fr3/visual/link4.dae
- link fr3_link5: geometry collision mesh filename=./assets/fr3/collision/link5.stl; visual mesh filename=./assets/fr3/visual/link5.dae
- link fr3_link6: geometry collision mesh filename=./assets/fr3/collision/link6.stl; visual mesh filename=./assets/fr3/visual/link6.dae
- link fr3_link7: geometry collision mesh filename=./assets/fr3/collision/link7.stl; visual mesh filename=./assets/fr3/visual/link7.dae
- link gripper_base_link: mass 0.18972 -> 0.4569787916
- link gripper_left_link: mass 0.033674 -> 0.0811106042
- link gripper_right_link: mass 0.033674 -> 0.0811106042
Joints:
- added joint fr3_pika_adapter_joint: type fixed, parent fr3_link8, child fr3_pika_adapter_link, origin xyz=-0.033 -0.033 -0.012 rpy=0 0 -0.
- added joint pika_task_tcp_joint: type fixed, parent gripper_base_link, child pika_task_tcp, origin xyz=0 0 0.366842 rpy=3.1415926 -1.5707963 0
- joint fr3_gripper_joint: origin xyz=0 0 0 rpy=-0.739815 -1.5707963 3.1415926 -> xyz=0.002 0 0.008 rpy=-0.739815 -1.5707963 3.1415926
- joint fr3_hand_tcp_joint: origin xyz=0.15 0 0.0285 rpy=3.1415926 -1.5707963 0 -> xyz=0.185 0 0 rpy=3.1415926 -1.5707963 0
