Commit message: feat: gate real replay on reviewed MuJoCo results

File: src/lerobot/robots/franka_research3/assets/franka_fr3/fr3_corenetic_gripper.urdf (robot description, URDF)
Before this commit: robot fr3_corenetic_gripper, 24 links, 23 joints
Links:
- added link fr3_ee
Joints:
- added joint fr3_ee_joint: type fixed, parent fr3_link8, child fr3_ee, origin xyz=0 0 0 rpy=0 0 0

Commit message: feat(fr3): align corenetic gripper description with v2 mesh set
Point fr3_corenetic_gripper.urdf/.xml at the new
gripper_w_v2_franka_description/ meshes (link_gripper_*, ft sensor
and tip links) and add the SMR-cam mount from corenetic_smr_cam/ as
a fixed child of the end-effector for the laser-tracker rig.

File: src/lerobot/robots/franka_research3/assets/franka_fr3/fr3_corenetic_gripper.urdf (robot description, URDF)
Before this commit: robot fr3_corenetic_gripper, 25 links, 24 joints
Links:
- removed link link_franka_corenetic_gripper_2
- removed link link_franka_corenetic_gripper_3
- removed link link_lt_gripper_base
- removed link link_lt_gripper_drive
- removed link link_lt_gripper_finger_left
- removed link link_lt_gripper_finger_right
- removed link link_lt_gripper_knuckle_left_inner
- removed link link_lt_gripper_knuckle_left_outer
- removed link link_lt_gripper_knuckle_right_inner
- removed link link_lt_gripper_knuckle_right_outer
- removed link link_lt_gripper_tcp
- added link link_corenetic_mount, mass 0.046529; collision mesh filename=corenetic_smr_cam/meshes/mount.STL; visual mesh filename=corenetic_smr_cam/meshes/mount.STL
- added link link_corenetic_smr, mass 0.14; collision sphere radius=0.01905; visual sphere radius=0.01905
- added link link_corenetic_smr_cam, mass 0.1871; collision mesh filename=corenetic_smr_cam/meshes/smr_cam_base.STL; collision mesh filename=corenetic_smr_cam/meshes/smr_cam_camera.STL
- added link link_gripper_base, mass 4.3437052889E-01; collision mesh filename=gripper_w_v2_franka_description/meshes/link_gripper_base.STL; visual mesh filename=gripper_w_v2_franka_description/meshes/link_gripper_base.STL
- added link link_gripper_contact_left
- added link link_gripper_contact_right
- added link link_gripper_drive
- added link link_gripper_finger_left, mass 1E-16; collision mesh filename=gripper_w_v2_franka_description/meshes/link_gripper_finger_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; visual mesh filename=gripper_w_v2_franka_description/meshes/link_gripper_finger_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
- added link link_gripper_finger_right, mass 1E-16; collision mesh filename=gripper_w_v2_franka_description/meshes/link_gripper_finger_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; visual mesh filename=gripper_w_v2_franka_description/meshes/link_gripper_finger_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
- added link link_gripper_knuckle_left_inner, mass 1E-16; collision mesh filename=gripper_w_v2_franka_description/meshes/link_gripper_knuckle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; visual mesh filename=gripper_w_v2_franka_description/meshes/link_gripper_knuckle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
- added link link_gripper_knuckle_left_outer, mass 1E-16; collision mesh filename=gripper_w_v2_franka_description/meshes/link_gripper_knuckle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; visual mesh filename=gripper_w_v2_franka_description/meshes/link_gripper_knuckle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
- added link link_gripper_knuckle_right_inner, mass 1E-16; collision mesh filename=gripper_w_v2_franka_description/meshes/link_gripper_knuckle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; visual mesh filename=gripper_w_v2_franka_description/meshes/link_gripper_knuckle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
- added link link_gripper_knuckle_right_outer, mass 1E-16; collision mesh filename=gripper_w_v2_franka_description/meshes/link_gripper_knuckle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; visual mesh filename=gripper_w_v2_franka_description/meshes/link_gripper_knuckle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
- added link link_gripper_tcp
- added link link_gripper_tip_left, mass 1E-16; collision mesh filename=gripper_w_v2_franka_description/meshes/link_gripper_tip_lef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; visual mesh filename=gripper_w_v2_franka_description/meshes/link_gripper_tip_lef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
- added link link_gripper_tip_right, mass 1E-16; collision mesh filename=gripper_w_v2_franka_description/meshes/link_gripper_tip_rig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; visual mesh filename=gripper_w_v2_franka_description/meshes/link_gripper_tip_rig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
- added link link_sensor_ft, mass 0.0525656216796275; collision mesh filename=gripper_w_v2_franka_description/meshes/link_sensor_ft.STL; visual mesh filename=gripper_w_v2_franka_description/meshes/link_sensor_ft.STL
- link base_link: mass 0.0280919165597075 -> 7.5848174710E-02; geometry collision mesh filename=gripper_w_v2_franka_description/meshes/base_link.STL; visual mesh filename=gripper_w_v2_franka_description/meshes/base_link.STL
- link link_franka_corenetic_gripper_1: geometry collision mesh filename=gripper_w_v2_franka_description/meshes/link_franka_coreneti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; visual mesh filename=gripper_w_v2_franka_description/meshes/link_franka_coreneti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
Joints:
- removed joint joint_franka_corenetic_gripper_2
- removed joint joint_franka_corenetic_gripper_3
- removed joint joint_lt_gripper_base
- removed joint joint_lt_gripper_drive
- removed joint joint_lt_gripper_finger_left
- removed joint joint_lt_gripper_finger_right
- removed joint joint_lt_gripper_knuckle_left_inner
- removed joint joint_lt_gripper_knuckle_left_outer
- removed joint joint_lt_gripper_knuckle_right_inner
- removed joint joint_lt_gripper_knuckle_right_outer
- removed joint joint_lt_gripper_tcp
- added joint joint_corenetic_mount: type fixed, parent base_link, child link_corenetic_mount, origin xyz=0 0 0 rpy=0 0 0
- added joint joint_corenetic_smr: type fixed, parent link_corenetic_smr_cam, child link_corenetic_smr, origin xyz=0.070201 -0.000249 0.103891 rpy=0 0 0
- added joint joint_corenetic_smr_cam: type fixed, parent link_corenetic_mount, child link_corenetic_smr_cam, origin xyz=0 0 0 rpy=0 0 0
- added joint joint_gripper_base: type fixed, parent link_sensor_ft, child link_gripper_base, origin xyz=0 0 0.01375 rpy=3.14159265358979 0 1.5707963267949, axis 0 0 0
- added joint joint_gripper_contact_left: type fixed, parent link_gripper_tip_left, child link_gripper_contact_left, origin xyz=0 -0.0115 -0.005 rpy=0 0 0, axis 0 0 0
- added joint joint_gripper_contact_right: type fixed, parent link_gripper_tip_right, child link_gripper_contact_right, origin xyz=0 0.0115 -0.005 rpy=0 0 0, axis 0 0 0
- added joint joint_gripper_drive: type revolute, parent link_gripper_base, child link_gripper_drive, origin xyz=0 0 0 rpy=0 0 0, axis 0 0 1, limit lower=0 upper=1.5708 effort=6 velocity=1.5708
- added joint joint_gripper_finger_left: type revolute, parent link_gripper_knuckle_left_outer, child link_gripper_finger_left, origin xyz=0 0.005475 -0.049699 rpy=0 0 0, axis -1 0 0, limit lower=0 upper=1.44339 effort=6 velocity=1.5708, mimic joint=joint_gripper_drive multiplier=1 offset=0
- added joint joint_gripper_finger_right: type revolute, parent link_gripper_knuckle_right_outer, child link_gripper_finger_right, origin xyz=0 -0.005475 -0.049699 rpy=0 0 0, axis 1 0 0, limit lower=0 upper=1.44339 effort=6 velocity=1.5708, mimic joint=joint_gripper_drive multiplier=1 offset=0
- added joint joint_gripper_knuckle_left_inner: type revolute, parent link_gripper_base, child link_gripper_knuckle_left_inner, origin xyz=0 0.0074298 -0.066289 rpy=0 0 0, axis 1 0 0, limit lower=0 upper=1.4434 effort=6 velocity=1.5708, mimic joint=joint_gripper_drive multiplier=1 offset=0
- added joint joint_gripper_knuckle_left_outer: type revolute, parent link_gripper_base, child link_gripper_knuckle_left_outer, origin xyz=0 0.019 -0.0525 rpy=0 0 0, axis 1 0 0, limit lower=0 upper=1.4434 effort=6 velocity=1.5708, mimic joint=joint_gripper_drive multiplier=1 offset=0
- added joint joint_gripper_knuckle_right_inner: type revolute, parent link_gripper_base, child link_gripper_knuckle_right_inner, origin xyz=0 -0.0074298 -0.066289 rpy=0 0 0, axis -1 0 0, limit lower=0 upper=1.4434 effort=6 velocity=1.5708, mimic joint=joint_gripper_drive multiplier=1 offset=0
- added joint joint_gripper_knuckle_right_outer: type revolute, parent link_gripper_base, child link_gripper_knuckle_right_outer, origin xyz=0 -0.019 -0.0525 rpy=0 0 0, axis -1 0 0, limit lower=0 upper=1.44339 effort=6 velocity=1.5708, mimic joint=joint_gripper_drive multiplier=1 offset=0
- added joint joint_gripper_tcp: type fixed, parent link_gripper_base, child link_gripper_tcp, origin xyz=0 0 -0.13599 rpy=3.1416 0 0, axis 0 0 0
- added joint joint_gripper_tip_left: type fixed, parent link_gripper_finger_left, child link_gripper_tip_left, origin xyz=0 -0.012975 -0.028789 rpy=0 0 0, axis 0 0 0
- added joint joint_gripper_tip_right: type fixed, parent link_gripper_finger_right, child link_gripper_tip_right, origin xyz=0 0.012975 -0.028789 rpy=0 0 0, axis 0 0 0
- added joint joint_sensor_ft: type fixed, parent base_link, child link_sensor_ft, origin xyz=0 0 0.02225 rpy=0 0 -1.57079632679492, axis 0 0 0
- joint fr3_hand_tcp_joint: origin xyz=0 0 -0.0 rpy=3.141592653589793 0 0 -> xyz=0 0 0 rpy=0 0 0; parent link_lt_gripper_tcp -> link_gripper_tcp

Commit message: feat(fr3): add link_lt_gripper_tcp compatibility frame for laser bundles
The marker->TCP bundles from the old URDF_franka_corenetic_gripper/
package were defined in its TCP axes (z toward the flange). Now that
the EE is a child of the v2 gripper's link_gripper_tcp, those bundles
no longer line up: the laser-tracker tracker and the replay both hop
R_x(pi) from the bundle frame to the EE. Hanging corenetic_gripper_ee
off a new link_lt_gripper_tcp (R_x(pi) from link_gripper_tcp) keeps
the old bundle origins valid. Rename the hop to link_gripper_tcp and
every EE orientation flips without an error.

File: src/lerobot/robots/franka_research3/assets/franka_fr3/fr3_corenetic_gripper.urdf (robot description, URDF)
Before this commit: robot fr3_corenetic_gripper, 31 links, 30 joints
Links:
- added link link_lt_gripper_tcp
Joints:
- added joint joint_lt_gripper_tcp: type fixed, parent link_gripper_tcp, child link_lt_gripper_tcp, origin xyz=0 0 0 rpy=3.141592653589793 0 0
- joint fr3_hand_tcp_joint: origin xyz=0 0 0 rpy=0 0 0 -> xyz=0 0 0 rpy=3.141592653589793 0 0; parent link_gripper_tcp -> link_lt_gripper_tcp

Commit message: feat(fr3): TCP pivot calibration + corenetic_socket_ee URDF frame
The camera EE trajectories put their TCP at the socket centre of
pivot insert v2; the FR3 was driving corenetic_gripper_ee (the
vendor closed-fingertip point, 171.99 mm below the flange). The
10-12 end-to-end replay saw a constant ~10 mm bias along the tool
axis between them, which the laser measures as the offset.

- lerobot.robots.franka_research3.tcp_pivot: pure-numpy fit of
  (s, c) from EE rotations while a point fixed to the tool stays
  on a fixed base point; orientation-bin subsampling and a
  time-block jackknife for sigma. Rejects a 0.5 mm lift-off in
  3 outer rounds and raises when the orientation spread does not
  observe s.
- tools/fr3/fr3_tcp_pivot.py: real-robot collect (teaching mode)
  and fit (pinocchio FK -> corenetic_gripper_ee), with the Desk
  O_T_EE fit as a cross-check.
- fr3_corenetic_gripper.urdf/.xml: add corenetic_socket_ee as a
  pure -z translation of corenetic_gripper_ee, the pivot insert's
  socket centre measured with the laser (10-12: -10.7, 10-13:
  -9.9 mm). Reject any rotation in the URDF contract; the camera
  labels the socket with EE axes.
- gripper_w_v2_franka_description/README.md: warn that the vendor
  finger meshes are 9 mm long on the tool axis, so they cannot
  locate the socket; the laser measurement is the only source.
- test_fr3_socket_frame.py: covers the URDF + replay/IK-QC
  contract (no rotation, parent is corenetic_gripper_ee).
- test_fr3_tcp_pivot.py: covers the math against an analytical
  sweep, the observability check, the lift-off reject, and the
  jackknife.
- cube_replay_ui.md: panel-level doc of the new target frame.
- Submodule: replay/IK-QC configs and the URDF contract in
  third_party/opencv_kalibr to drive corenetic_socket_ee.

File: src/lerobot/robots/franka_research3/assets/franka_fr3/fr3_corenetic_gripper.urdf (robot description, URDF)
Before this commit: robot fr3_corenetic_gripper, 32 links, 31 joints
Links:
- added link corenetic_socket_ee
Joints:
- added joint corenetic_socket_joint: type fixed, parent corenetic_gripper_ee, child corenetic_socket_ee, origin xyz=0 0 -0.0103 rpy=0 0 0
