Commit message: calib(fr3): corenetic_socket_ee from the FR3 pivot, (1.45, -0.78, -5.06) mm
Nine runs about a fixed ball fitted together (sigma <= 0.35 mm, leave one run
out <= 0.36 mm); a caliper reads flange face -> socket 166.9 mm. The earlier
z -10.3 mm was fitted end to end with the laser and had absorbed about 5 mm of
the world -> fr3_base edge's error along the tool axis. Bumps opencv_kalibr
for the matching config comments.

Co-Authored-By: Claude Opus 5.5 <noreply@anthropic.com>

File: src/lerobot/robots/franka_research3/assets/franka_fr3/fr3_corenetic_gripper.urdf (robot description, URDF)
Before this commit: robot fr3_corenetic_gripper, 33 links, 32 joints
Joints:
- joint corenetic_socket_joint: origin xyz=0 0 -0.0103 rpy=0 0 0 -> xyz=0.00145 -0.00078 -0.00506 rpy=0 0 0

Commit message: feat(fr3/thor): fr3_base registration edge, FR3 laser replay and pivot calibration
Squash of hph/fr3_base_registration_edge (2026-10-09 .. 10-15, 56 commits,
supersedes #51 and #52) onto box.

World / registration
- Register the FR3 base as a world-graph edge; export_v3 --target-world
  re-expresses labels in fr3_base (default for FR3 export/deploy).
- Keep EE trajectories on the 0928 world after #50 (world_provenance).
- world -> fr3_base edge via the laser tracker (register_fr3_base.py) and via
  the FR3 / handheld same-ball check (fr3_base_ball_check.py); production edge
  is the 5-position ball edge ball_check_20261015T030840Z (leave-one-out
  rms 2.63 mm).
- Production calibration calib_20261014_180431, world W kept by registering
  on camera centres.

FR3 replay and calibration
- Two-step real replay on Thor with optional laser-tracker recording; replays
  the recorded gripper / BOX trigger; start pose planned inside panda_py's
  joint wall; command lead (default 3 frames); move-to-start button.
- Payload identification library + runtime (Desk load set from measurement).
- Gripper description switched to the vendor v2 mesh set; corenetic_smr_cam
  assets; link_lt_gripper_tcp compatibility frame; corenetic_socket_ee frame
  from the FR3 pivot (1.45, -0.78, -5.06) mm.
- TCP pivot calibration, ball pivot joint fit, guided / planned pivot with
  wall checks, dwell planner over a surveyed feasible set.
- Handheld BOX drives the FR3 gripper BOX; BOX gripper addressed by device_id
  and re-taken after a mid-replay restart.

Data / timing
- BOX data paired at the camera's mid-exposure plus a per-BOX transport delay
  (box_time_delays.json, box_realign.py).
- Laser tracker episode gate + verdict banner; StartEpisode blocked when the
  tracker is in error or the beam is on its home nest.

GUI
- Laser replay analysis panel, calibration-page panels for FR3 pivot, gripper
  teleop and laser / ball edges, camera state per recording.

Submodules: opencv_kalibr -> bb594440 (FR3 replay laser-error evaluator,
corenetic_socket_ee drive); box_sdk -> 1c2520c (pinned device_id,
keep_mode_device_ids).

Docs: GT roadmaps v1.14-v1.27, payload identification report, 3 mm stage
summary, 10-12 - 10-15 weekly report.

Co-Authored-By: Claude Opus 5.5 <noreply@anthropic.com>

File: src/lerobot/robots/franka_research3/assets/franka_fr3/fr3_corenetic_gripper.urdf (robot description, URDF)
Before this commit: robot fr3_corenetic_gripper, 25 links, 24 joints
Links:
- removed link link_franka_corenetic_gripper_2
- removed link link_franka_corenetic_gripper_3
- removed link link_lt_gripper_base
- removed link link_lt_gripper_drive
- removed link link_lt_gripper_finger_left
- removed link link_lt_gripper_finger_right
- removed link link_lt_gripper_knuckle_left_inner
- removed link link_lt_gripper_knuckle_left_outer
- removed link link_lt_gripper_knuckle_right_inner
- removed link link_lt_gripper_knuckle_right_outer
- added link corenetic_socket_ee
- added link link_corenetic_mount, mass 0.046529; collision mesh filename=corenetic_smr_cam/meshes/mount.STL; visual mesh filename=corenetic_smr_cam/meshes/mount.STL
- added link link_corenetic_smr, mass 0.14; collision sphere radius=0.01905; visual sphere radius=0.01905
- added link link_corenetic_smr_cam, mass 0.1871; collision mesh filename=corenetic_smr_cam/meshes/smr_cam_base.STL; collision mesh filename=corenetic_smr_cam/meshes/smr_cam_camera.STL
- added link link_gripper_base, mass 4.3437052889E-01; collision mesh filename=gripper_w_v2_franka_description/meshes/link_gripper_base.STL; visual mesh filename=gripper_w_v2_franka_description/meshes/link_gripper_base.STL
- added link link_gripper_contact_left
- added link link_gripper_contact_right
- added link link_gripper_drive
- added link link_gripper_finger_left, mass 1E-16; collision mesh filename=gripper_w_v2_franka_description/meshes/link_gripper_finger_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; visual mesh filename=gripper_w_v2_franka_description/meshes/link_gripper_finger_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
- added link link_gripper_finger_right, mass 1E-16; collision mesh filename=gripper_w_v2_franka_description/meshes/link_gripper_finger_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; visual mesh filename=gripper_w_v2_franka_description/meshes/link_gripper_finger_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
- added link link_gripper_knuckle_left_inner, mass 1E-16; collision mesh filename=gripper_w_v2_franka_description/meshes/link_gripper_knuckle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; visual mesh filename=gripper_w_v2_franka_description/meshes/link_gripper_knuckle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
- added link link_gripper_knuckle_left_outer, mass 1E-16; collision mesh filename=gripper_w_v2_franka_description/meshes/link_gripper_knuckle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; visual mesh filename=gripper_w_v2_franka_description/meshes/link_gripper_knuckle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
- added link link_gripper_knuckle_right_inner, mass 1E-16; collision mesh filename=gripper_w_v2_franka_description/meshes/link_gripper_knuckle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; visual mesh filename=gripper_w_v2_franka_description/meshes/link_gripper_knuckle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
- added link link_gripper_knuckle_right_outer, mass 1E-16; collision mesh filename=gripper_w_v2_franka_description/meshes/link_gripper_knuckle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; visual mesh filename=gripper_w_v2_franka_description/meshes/link_gripper_knuckle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
- added link link_gripper_tcp
- added link link_gripper_tip_left, mass 1E-16; collision mesh filename=gripper_w_v2_franka_description/meshes/link_gripper_tip_lef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; visual mesh filename=gripper_w_v2_franka_description/meshes/link_gripper_tip_lef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
- added link link_gripper_tip_right, mass 1E-16; collision mesh filename=gripper_w_v2_franka_description/meshes/link_gripper_tip_rig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; visual mesh filename=gripper_w_v2_franka_description/meshes/link_gripper_tip_rig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
- added link link_sensor_ft, mass 0.0525656216796275; collision mesh filename=gripper_w_v2_franka_description/meshes/link_sensor_ft.STL; visual mesh filename=gripper_w_v2_franka_description/meshes/link_sensor_ft.STL
- link base_link: mass 0.0280919165597075 -> 7.5848174710E-02; geometry collision mesh filename=gripper_w_v2_franka_description/meshes/base_link.STL; visual mesh filename=gripper_w_v2_franka_description/meshes/base_link.STL
- link link_franka_corenetic_gripper_1: geometry collision mesh filename=gripper_w_v2_franka_description/meshes/link_franka_coreneti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; visual mesh filename=gripper_w_v2_franka_description/meshes/link_franka_coreneti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
Joints:
- removed joint joint_franka_corenetic_gripper_2
- removed joint joint_franka_corenetic_gripper_3
- removed joint joint_lt_gripper_base
- removed joint joint_lt_gripper_drive
- removed joint joint_lt_gripper_finger_left
- removed joint joint_lt_gripper_finger_right
- removed joint joint_lt_gripper_knuckle_left_inner
- removed joint joint_lt_gripper_knuckle_left_outer
- removed joint joint_lt_gripper_knuckle_right_inner
- removed joint joint_lt_gripper_knuckle_right_outer
- added joint corenetic_socket_joint: type fixed, parent corenetic_gripper_ee, child corenetic_socket_ee, origin xyz=0.00145 -0.00078 -0.00506 rpy=0 0 0
- added joint joint_corenetic_mount: type fixed, parent base_link, child link_corenetic_mount, origin xyz=0 0 0 rpy=0 0 0
- added joint joint_corenetic_smr: type fixed, parent link_corenetic_smr_cam, child link_corenetic_smr, origin xyz=0.070201 -0.000249 0.103891 rpy=0 0 0
- added joint joint_corenetic_smr_cam: type fixed, parent link_corenetic_mount, child link_corenetic_smr_cam, origin xyz=0 0 0 rpy=0 0 0
- added joint joint_gripper_base: type fixed, parent link_sensor_ft, child link_gripper_base, origin xyz=0 0 0.01375 rpy=3.14159265358979 0 1.5707963267949, axis 0 0 0
- added joint joint_gripper_contact_left: type fixed, parent link_gripper_tip_left, child link_gripper_contact_left, origin xyz=0 -0.0115 -0.005 rpy=0 0 0, axis 0 0 0
- added joint joint_gripper_contact_right: type fixed, parent link_gripper_tip_right, child link_gripper_contact_right, origin xyz=0 0.0115 -0.005 rpy=0 0 0, axis 0 0 0
- added joint joint_gripper_drive: type revolute, parent link_gripper_base, child link_gripper_drive, origin xyz=0 0 0 rpy=0 0 0, axis 0 0 1, limit lower=0 upper=1.5708 effort=6 velocity=1.5708
- added joint joint_gripper_finger_left: type revolute, parent link_gripper_knuckle_left_outer, child link_gripper_finger_left, origin xyz=0 0.005475 -0.049699 rpy=0 0 0, axis -1 0 0, limit lower=0 upper=1.44339 effort=6 velocity=1.5708, mimic joint=joint_gripper_drive multiplier=1 offset=0
- added joint joint_gripper_finger_right: type revolute, parent link_gripper_knuckle_right_outer, child link_gripper_finger_right, origin xyz=0 -0.005475 -0.049699 rpy=0 0 0, axis 1 0 0, limit lower=0 upper=1.44339 effort=6 velocity=1.5708, mimic joint=joint_gripper_drive multiplier=1 offset=0
- added joint joint_gripper_knuckle_left_inner: type revolute, parent link_gripper_base, child link_gripper_knuckle_left_inner, origin xyz=0 0.0074298 -0.066289 rpy=0 0 0, axis 1 0 0, limit lower=0 upper=1.4434 effort=6 velocity=1.5708, mimic joint=joint_gripper_drive multiplier=1 offset=0
- added joint joint_gripper_knuckle_left_outer: type revolute, parent link_gripper_base, child link_gripper_knuckle_left_outer, origin xyz=0 0.019 -0.0525 rpy=0 0 0, axis 1 0 0, limit lower=0 upper=1.4434 effort=6 velocity=1.5708, mimic joint=joint_gripper_drive multiplier=1 offset=0
- added joint joint_gripper_knuckle_right_inner: type revolute, parent link_gripper_base, child link_gripper_knuckle_right_inner, origin xyz=0 -0.0074298 -0.066289 rpy=0 0 0, axis -1 0 0, limit lower=0 upper=1.4434 effort=6 velocity=1.5708, mimic joint=joint_gripper_drive multiplier=1 offset=0
- added joint joint_gripper_knuckle_right_outer: type revolute, parent link_gripper_base, child link_gripper_knuckle_right_outer, origin xyz=0 -0.019 -0.0525 rpy=0 0 0, axis -1 0 0, limit lower=0 upper=1.44339 effort=6 velocity=1.5708, mimic joint=joint_gripper_drive multiplier=1 offset=0
- added joint joint_gripper_tcp: type fixed, parent link_gripper_base, child link_gripper_tcp, origin xyz=0 0 -0.13599 rpy=3.1416 0 0, axis 0 0 0
- added joint joint_gripper_tip_left: type fixed, parent link_gripper_finger_left, child link_gripper_tip_left, origin xyz=0 -0.012975 -0.028789 rpy=0 0 0, axis 0 0 0
- added joint joint_gripper_tip_right: type fixed, parent link_gripper_finger_right, child link_gripper_tip_right, origin xyz=0 0.012975 -0.028789 rpy=0 0 0, axis 0 0 0
- added joint joint_sensor_ft: type fixed, parent base_link, child link_sensor_ft, origin xyz=0 0 0.02225 rpy=0 0 -1.57079632679492, axis 0 0 0
- joint fr3_hand_tcp_joint: origin xyz=0 0 -0.0 rpy=3.141592653589793 0 0 -> xyz=0 0 0 rpy=3.141592653589793 0 0
- joint joint_lt_gripper_tcp: axis 0 0 0 -> (none); origin xyz=0 0 -0.155 rpy=0 0 0 -> xyz=0 0 0 rpy=3.141592653589793 0 0; parent link_lt_gripper_base -> link_gripper_tcp

File: src/lerobot/robots/franka_research3/assets/franka_fr3/gripper_w_v2_franka_description/urdf/gripper_w_v2_franka_description.urdf (robot description, URDF)
Before this commit: robot URDF_franka_corenetic_gripper, 13 links, 13 joints
Links:
- removed link link_franka_corenetic_gripper_2
- removed link link_lt_gripper_base
- removed link link_lt_gripper_drive
- removed link link_lt_gripper_finger_left
- removed link link_lt_gripper_finger_right
- removed link link_lt_gripper_knuckle_left_inner
- removed link link_lt_gripper_knuckle_left_outer
- removed link link_lt_gripper_knuckle_right_inner
- removed link link_lt_gripper_knuckle_right_outer
- removed link link_lt_gripper_tcp
- added link link_gripper_base, mass 4.3437052889E-01; collision mesh filename=../meshes/collision/link_gripper_base.STL; visual mesh filename=../meshes/visual/link_gripper_base.STL
- added link link_gripper_contact_left
- added link link_gripper_contact_right
- added link link_gripper_drive
- added link link_gripper_finger_left, mass 1E-16; visual mesh filename=../meshes/visual/link_gripper_finger_left.STL
- added link link_gripper_finger_right, mass 1E-16; visual mesh filename=../meshes/visual/link_gripper_finger_right.STL
- added link link_gripper_knuckle_left_inner, mass 1E-16; visual mesh filename=../meshes/visual/link_gripper_knuckle_left_inner.STL
- added link link_gripper_knuckle_left_outer, mass 1E-16; visual mesh filename=../meshes/visual/link_gripper_knuckle_left_outer.STL
- added link link_gripper_knuckle_right_inner, mass 1E-16; visual mesh filename=../meshes/visual/link_gripper_knuckle_right_inner.STL
- added link link_gripper_knuckle_right_outer, mass 1E-16; visual mesh filename=../meshes/visual/link_gripper_knuckle_right_outer.STL
- added link link_gripper_tcp
- added link link_gripper_tip_left, mass 1E-16; visual mesh filename=../meshes/visual/link_gripper_tip_left.STL
- added link link_gripper_tip_right, mass 1E-16; visual mesh filename=../meshes/visual/link_gripper_tip_right.STL
- added link link_sensor_ft, mass 0.0525656216796275; collision mesh filename=../meshes/collision/link_sensor_ft.STL; visual mesh filename=../meshes/visual/link_sensor_ft.STL
- link base_link: mass 0.0280919165597075 -> 7.5848174710E-02; geometry collision mesh filename=../meshes/collision/base_link.STL; visual mesh filename=../meshes/visual/base_link.STL
- link link_franka_corenetic_gripper_1: geometry collision mesh filename=../meshes/collision/link_franka_corenetic_gripper_1.STL; visual mesh filename=../meshes/visual/link_franka_corenetic_gripper_1.STL
- link link_franka_corenetic_gripper_3: geometry collision mesh filename=../meshes/collision/link_franka_corenetic_gripper_3.STL; visual mesh filename=../meshes/visual/link_franka_corenetic_gripper_3.STL
Joints:
- removed joint joint_franka_corenetic_gripper_2
- removed joint joint_lt_gripper_drive
- removed joint joint_lt_gripper_finger_left
- removed joint joint_lt_gripper_finger_right
- removed joint joint_lt_gripper_knuckle_left_inner
- removed joint joint_lt_gripper_knuckle_left_outer
- removed joint joint_lt_gripper_knuckle_right_inner
- removed joint joint_lt_gripper_knuckle_right_outer
- removed joint joint_lt_gripper_tcp
- added joint joint_gripper_base: type fixed, parent link_sensor_ft, child link_gripper_base, origin xyz=0 0 0.01375 rpy=3.14159265358979 0 1.5707963267949, axis 0 0 0
- added joint joint_gripper_contact_left: type fixed, parent link_gripper_tip_left, child link_gripper_contact_left, origin xyz=0 -0.0115 -0.005 rpy=0 0 0, axis 0 0 0
- added joint joint_gripper_contact_right: type fixed, parent link_gripper_tip_right, child link_gripper_contact_right, origin xyz=0 0.0115 -0.005 rpy=0 0 0, axis 0 0 0
- added joint joint_gripper_drive: type revolute, parent link_gripper_base, child link_gripper_drive, origin xyz=0 0 0 rpy=0 0 0, axis 0 0 1, limit lower=0 upper=1.5708 effort=6 velocity=1.5708
- added joint joint_gripper_finger_left: type revolute, parent link_gripper_knuckle_left_outer, child link_gripper_finger_left, origin xyz=0 0.005475 -0.049699 rpy=0 0 0, axis -1 0 0, limit lower=0 upper=1.44339 effort=6 velocity=1.5708, mimic joint=joint_gripper_drive multiplier=1 offset=0
- added joint joint_gripper_finger_right: type revolute, parent link_gripper_knuckle_right_outer, child link_gripper_finger_right, origin xyz=0 -0.005475 -0.049699 rpy=0 0 0, axis 1 0 0, limit lower=0 upper=1.44339 effort=6 velocity=1.5708, mimic joint=joint_gripper_drive multiplier=1 offset=0
- added joint joint_gripper_knuckle_left_inner: type revolute, parent link_gripper_base, child link_gripper_knuckle_left_inner, origin xyz=0 0.0074298 -0.066289 rpy=0 0 0, axis 1 0 0, limit lower=0 upper=1.4434 effort=6 velocity=1.5708, mimic joint=joint_gripper_drive multiplier=1 offset=0
- added joint joint_gripper_knuckle_left_outer: type revolute, parent link_gripper_base, child link_gripper_knuckle_left_outer, origin xyz=0 0.019 -0.0525 rpy=0 0 0, axis 1 0 0, limit lower=0 upper=1.4434 effort=6 velocity=1.5708, mimic joint=joint_gripper_drive multiplier=1 offset=0
- added joint joint_gripper_knuckle_right_inner: type revolute, parent link_gripper_base, child link_gripper_knuckle_right_inner, origin xyz=0 -0.0074298 -0.066289 rpy=0 0 0, axis -1 0 0, limit lower=0 upper=1.4434 effort=6 velocity=1.5708, mimic joint=joint_gripper_drive multiplier=1 offset=0
- added joint joint_gripper_knuckle_right_outer: type revolute, parent link_gripper_base, child link_gripper_knuckle_right_outer, origin xyz=0 -0.019 -0.0525 rpy=0 0 0, axis -1 0 0, limit lower=0 upper=1.44339 effort=6 velocity=1.5708, mimic joint=joint_gripper_drive multiplier=1 offset=0
- added joint joint_gripper_tcp: type fixed, parent link_gripper_base, child link_gripper_tcp, origin xyz=0 0 -0.13599 rpy=3.1416 0 0, axis 0 0 0
- added joint joint_gripper_tip_left: type fixed, parent link_gripper_finger_left, child link_gripper_tip_left, origin xyz=0 -0.012975 -0.028789 rpy=0 0 0, axis 0 0 0
- added joint joint_gripper_tip_right: type fixed, parent link_gripper_finger_right, child link_gripper_tip_right, origin xyz=0 0.012975 -0.028789 rpy=0 0 0, axis 0 0 0
- added joint joint_sensor_ft: type fixed, parent base_link, child link_sensor_ft, origin xyz=0 0 0.02225 rpy=0 0 -1.57079632679492, axis 0 0 0
